File: shield/shield.sch (KiCad schematic (older format))
At the start: 16 parts, among them J1 Screw_Terminal_1x04, J2 Screw_Terminal_1x02, J3 CONN_01X04, J4 Screw_Terminal_1x06, P1 CONN_01X08, P2 CONN_01X08, Q1 Q_NMOS_GDS, Q2 Q_NMOS_GDS, Q3 Q_NMOS_GDS, SW1 Rotary_Encoder_Switch

Commit message: Modified the shield design to utilise a 3V3 LDO instead of 5V regulator module. Powering the Wemos D1 Mini through it's 3V3 pin instead of 5V (effectively bypassing the onboard regulator).
Parts:
- removed J3: CONN_01X04, symbol CONN_01X04
- added C3: 22uF, symbol C
- added U1: LM1117-3.3, symbol LM1117-3.3
Connections:
- net +12V: now also U1.3 (VI)
- net +3V3: now also C3.1, U1.2 (VO), U1.4 (VO)
- net GND: now also C3.2, U1.1 (GND/ADJ)
Other:
- note added: "3V3 regulator"
- note removed: "5V buck boost regulator"
- moved on the sheet: C1, D1, J2

Commit message: Schematic changes as per merge request discussion, and beginning PCB layout
Changes:
* Schematic
 * Changed rotary encoder schematic part
 * Added debounce circuitry to all rotary encoder signal lines
 * Changed rotary encoder pinout to match existing circuitry
 * Changed MOSFETs to GSD style
 * Added footprints for all components (ensuring hand solderability of all components)
* Library
 * Added custom footprints library for modified footprints / additional ones required
 * Added '3d' folder for attaching 3D bodies to components
* PCB
 * Initial placement of PCB completed
 * Removed pin names from bottom side silk screen
Parts:
- removed SW1: Rotary_Encoder_Switch, symbol Rotary_Encoder_Switch
- added C4, C5: 100nF, Capacitors_SMD:C_0805_HandSoldering, symbol C
- added R4, R5, R6: 27k, Resistors_SMD:R_0805_HandSoldering, symbol R
- added ROT1: ROTARY-ENCODER, sparkfun:SF-ROTARY-ENCODER, symbol ROTARY-ENCODER
- C1, C2, C3: footprint (none) -> Capacitors_SMD:C_0805_HandSoldering
- D1: footprint (none) -> Diodes_SMD:D_SMB-SMC_Universal_Handsoldering
- J1: footprint (none) -> Connectors_Terminal_Blocks:TerminalBlock_Pheonix_MPT-2.54mm_4pol
- J2: footprint (none) -> Connectors_Terminal_Blocks:TerminalBlock_Pheonix_MPT-2.54mm_2pol
- J4: footprint (none) -> Connectors_Terminal_Blocks:TerminalBlock_Pheonix_MPT-2.54mm_6pol
- Q1, Q2, Q3: value Q_NMOS_GDS -> Q_NMOS_GSD; footprint (none) -> TO_SOT_Packages_SMD:SOT-23_Handsoldering; symbol Q_NMOS_GDS -> Q_NMOS_GSD
- R1, R2, R3: footprint (none) -> Resistors_SMD:R_0805_HandSoldering
- U1: footprint (none) -> TO_SOT_Packages_SMD:SOT-223
Connections:
- net ENC_A: now also R4.1, ROT1.2 (A); no longer P1.5 (P5)
- net ENC_SWITCH: now also R6.2, ROT1.1 (SW1); no longer C2.1, P1.3 (P3)
- net GND: now also Q1.2 (S), Q2.2 (S), Q3.2 (S), C4.2, C5.2, ROT1.3 (C), ROT1.5 (SW2); no longer Q1.3 (S), Q2.3 (S), Q3.3 (S)
- net at J4.2: now also Q1.3 (D); no longer Q1.2 (D)
- net at J4.4: now also Q2.3 (D); no longer Q2.2 (D)
- net at J4.6: now also Q3.3 (D); no longer Q3.2 (D)
- net ENC_COM renamed MCU_A
- net MCU_A: now also C4.1, R4.2
- new net ENC_B: R5.1, ROT1.4 (B)
- new net MCU_B: C5.1, P1.5 (P5), R5.2
- new net MCU_SWITCH: C2.1, P1.3 (P3), R6.1
Other:
- moved on the sheet: C2
Changed lines of the file:
@@
 LIBS:contrib
 LIBS:valves
+LIBS:sparkfun
 LIBS:shield-cache
 EELAYER 25 0
@@
 Title "LED Strip Driver WeMos D1 Mini Shield"
 Date "2017-06-05"
-Rev "0.1"
+Rev "0.2"
 Comp ""
 Comment1 ""
@@
 F 0 "J2" H 1400 1950 50  0000 C TNN
 F 1 "Screw_Terminal_1x02" V 1250 1700 50  0000 C TNN
-F 2 "" H 1400 1475 50  0001 C CNN
+F 2 "Connectors_Terminal_Blocks:TerminalBlock_Pheonix_MPT-2.54mm_2pol" H 1400 1475 50  0001 C CNN
 F 3 "" H 1375 1700 50  0001 C CNN
 	1    1400 1700
@@
 F 0 "D1" H 1950 1700 50  0000 C CNN
 F 1 "D" H 1950 1500 50  0000 C CNN
-F 2 "" H 1950 1600 50  0001 C CNN
+F 2 "Diodes_SMD:D_SMB-SMC_Universal_Handsoldering" H 1950 1600 50  0001 C CNN
 F 3 "" H 1950 1600 50  0001 C CNN
 	1    1950 1600
@@
 F 0 "C1" H 2525 1800 50  0000 L CNN
 F 1 "10uF" H 2525 1600 50  0000 L CNN
-F 2 "" H 2538 1550 50  0001 C CNN
+F 2 "Capacitors_SMD:C_0805_HandSoldering" H 2538 1550 50  0001 C CNN
 F 3 "" H 2500 1700 50  0001 C CNN
 	1    2500 1700
@@
 Text Notes 1650 1200 0    60   ~ 0
 12V in
-$Comp
-L Rotary_Encoder_Switch SW1
-U 1 1 593540EC
-P 5700 5600
-F 0 "SW1" H 5700 5860 50  0000 C CNN
-F 1 "Rotary_Encoder_Switch" H 5700 5340 50  0000 C CNN
-F 2 "" H 5600 5760 50  0001 C CNN
-F 3 "" H 5700 5860 50  0001 C CNN
-	1    5700 5600
-	1    0    0    -1
-$EndComp
 $Comp
 L GND #PWR05
@@
 	1    0    0    -1
 $EndComp
-Text Label 6050 5500 0    60   ~ 0
+Text Label 6100 5500 0    60   ~ 0
 ENC_SWITCH
 $Comp
@@
 $EndComp
 Text Label 4700 5500 0    60   ~ 0
-ENC_COM
-Text Label 4700 5600 0    60   ~ 0
 ENC_A
 $Comp
@@
 F 0 "J1" H 1350 4550 50  0000 C TNN
 F 1 "Screw_Terminal_1x04" V 1200 4100 50  0000 C TNN
-F 2 "" H 1350 3675 50  0001 C CNN
+F 2 "Connectors_Terminal_Blocks:TerminalBlock_Pheonix_MPT-2.54mm_4pol" H 1350 3675 50  0001 C CNN
 F 3 "" H 1325 4300 50  0001 C CNN
 	1    1350 4100
@@
 F 0 "R1" V 9080 1600 50  0000 C CNN
 F 1 "220R" V 9000 1600 50  0000 C CNN
-F 2 "" V 8930 1600 50  0001 C CNN
+F 2 "Resistors_SMD:R_0805_HandSoldering" V 8930 1600 50  0001 C CNN
 F 3 "" H 9000 1600 50  0001 C CNN
 	1    9000 1600
@@
 $EndComp
 $Comp
-L Q_NMOS_GDS Q1
+L Q_NMOS_GSD Q1
 U 1 1 593565E4
 P 9000 2050
 F 0 "Q1" H 9200 2100 50  0000 L CNN
-F 1 "Q_NMOS_GDS" H 9200 2000 50  0000 L CNN
-F 2 "" H 9200 2150 50  0001 C CNN
+F 1 "Q_NMOS_GSD" H 9200 2000 50  0000 L CNN
+F 2 "TO_SOT_Packages_SMD:SOT-23_Handsoldering" H 9200 2150 50  0001 C CNN
 F 3 "" H 9000 2050 50  0001 C CNN
 	1    9000 2050
@@
 F 0 "R2" V 9080 3300 50  0000 C CNN
 F 1 "220R" V 9000 3300 50  0000 C CNN
-F 2 "" V 8930 3300 50  0001 C CNN
+F 2 "Resistors_SMD:R_0805_HandSoldering" V 8930 3300 50  0001 C CNN
 F 3 "" H 9000 3300 50  0001 C CNN
 	1    9000 3300
@@
 $EndComp
 $Comp
-L Q_NMOS_GDS Q2
+L Q_NMOS_GSD Q2
 U 1 1 59356DEC
 P 9000 3750
 F 0 "Q2" H 9200 3800 50  0000 L CNN
-F 1 "Q_NMOS_GDS" H 9200 3700 50  0000 L CNN
-F 2 "" H 9200 3850 50  0001 C CNN
+F 1 "Q_NMOS_GSD" H 9200 3700 50  0000 L CNN
+F 2 "TO_SOT_Packages_SMD:SOT-23_Handsoldering" H 9200 3850 50  0001 C CNN
 F 3 "" H 9000 3750 50  0001 C CNN
 	1    9000 3750
@@
 F 0 "R3" V 9080 4900 50  0000 C CNN
 F 1 "220R" V 9000 4900 50  0000 C CNN
-F 2 "" V 8930 4900 50  0001 C CNN
+F 2 "Resistors_SMD:R_0805_HandSoldering" V 8930 4900 50  0001 C CNN
 F 3 "" H 9000 4900 50  0001 C CNN
 	1    9000 4900
@@
 $EndComp
 $Comp
-L Q_NMOS_GDS Q3
+L Q_NMOS_GSD Q3
 U 1 1 59357023
 P 9000 5350
 F 0 "Q3" H 9200 5400 50  0000 L CNN
-F 1 "Q_NMOS_GDS" H 9200 5300 50  0000 L CNN
-F 2 "" H 9200 5450 50  0001 C CNN
+F 1 "Q_NMOS_GSD" H 9200 5300 50  0000 L CNN
+F 2 "TO_SOT_Packages_SMD:SOT-23_Handsoldering" H 9200 5450 50  0001 C CNN
 F 3 "" H 9000 5350 50  0001 C CNN
 	1    9000 5350
@@
 L C C2
 U 1 1 5935871D
-P 6700 5750
-F 0 "C2" H 6725 5850 50  0000 L CNN
-F 1 "100nF" H 6725 5650 50  0000 L CNN
-F 2 "" H 6738 5600 50  0001 C CNN
-F 3 "" H 6700 5750 50  0001 C CNN
-	1    6700 5750
+P 7250 5750
+F 0 "C2" H 7275 5850 50  0000 L CNN
+F 1 "100nF" H 7275 5650 50  0000 L CNN
+F 2 "Capacitors_SMD:C_0805_HandSoldering" H 7288 5600 50  0001 C CNN
+F 3 "" H 7250 5750 50  0001 C CNN
+	1    7250 5750
 	1    0    0    -1
 $EndComp
@@
 L GND #PWR015
 U 1 1 593587A2
-P 6700 6000
-F 0 "#PWR015" H 6700 5750 50  0001 C CNN
-F 1 "GND" H 6700 5850 50  0000 C CNN
-F 2 "" H 6700 6000 50  0001 C CNN
-F 3 "" H 6700 6000 50  0001 C CNN
-	1    6700 6000
+P 7250 6000
+F 0 "#PWR015" H 7250 5750 50  0001 C CNN
+F 1 "GND" H 7250 5850 50  0000 C CNN
+F 2 "" H 7250 6000 50  0001 C CNN
+F 3 "" H 7250 6000 50  0001 C CNN
+	1    7250 6000
 	1    0    0    -1
 $EndComp
 Text Notes 1400 3300 0    60   ~ 0
 General I/O
-Text Notes 5000 5100 0    60   ~ 0
+Text Notes 5100 5100 0    60   ~ 0
 Rotary encoder with switch
 Text Label 4000 3200 0    60   ~ 0
-ENC_SWITCH
-Text Label 4000 3400 0    60   ~ 0
-ENC_A
-Text Label 4000 3500 0    60   ~ 0
-ENC_COM
+MCU_SWITCH
 Text Notes 4800 3500 0    60   ~ 0
 D1
@@
 F 0 "J4" H 10650 4400 50  0000 C TNN
 F 1 "Screw_Terminal_1x06" V 10500 3750 50  0000 C TNN
-F 2 "" H 10650 3125 50  0001 C CNN
+F 2 "Connectors_Terminal_Blocks:TerminalBlock_Pheonix_MPT-2.54mm_6pol" H 10650 3125 50  0001 C CNN
 F 3 "" H 10625 4150 50  0001 C CNN
 	1    10650 3750
@@
 Connection ~ 2400 1950
 Wire Wire Line
-	6000 5700 6300 5700
-Wire Wire Line
 	6300 5700 6300 5800
 Wire Wire Line
-	5100 5800 5100 5700
-Wire Wire Line
-	5100 5700 5400 5700
-Wire Wire Line
-	3500 5500 5400 5500
-Wire Wire Line
-	3400 5600 5400 5600
+	5100 5600 5100 5800
 Wire Wire Line
 	1700 4550 1700 4400
@@
 	9400 5250 9400 5050
 Wire Wire Line
-	6700 6000 6700 5900
-Wire Wire Line
-	6700 5600 6700 5500
-Connection ~ 6700 5500
-Wire Wire Line
-	6000 5500 6800 5500
-Wire Wire Line
 	3700 3200 4950 3200
 Wire Wire Line
-	3400 3400 4950 3400
-Wire Wire Line
-	3500 3500 4950 3500
+	3200 3400 4950 3400
+Wire Wire Line
+	3400 3500 4950 3500
 Wire Wire Line
 	6450 3100 7400 3100
@@
 	6450 3500 6650 3500
 Wire Wire Line
-	3500 3500 3500 5500
-Wire Wire Line
-	3400 5600 3400 3400
-Wire Wire Line
 	2900 3300 2900 4200
-Wire Wire Line
-	3700 3200 3700 5300
-Wire Wire Line
-	3700 5300 6800 5300
-Wire Wire Line
-	6800 5300 6800 5500
 Wire Wire Line
 	1550 4000 2700 4000
@@
 F 0 "U1" H 3100 1200 50  0000 C CNN
 F 1 "LM1117-3.3" H 3000 1700 50  0000 C CNN
-F 2 "" H 3000 1450 50  0001 C CNN
+F 2 "TO_SOT_Packages_SMD:SOT-223" H 3000 1450 50  0001 C CNN
 F 3 "" H 3000 1450 50  0001 C CNN
 	1    3000 1450
@@
 F 0 "C3" H 3475 1800 50  0000 L CNN
 F 1 "22uF" H 3475 1600 50  0000 L CNN
-F 2 "" H 3488 1550 50  0001 C CNN
+F 2 "Capacitors_SMD:C_0805_HandSoldering" H 3488 1550 50  0001 C CNN
 F 3 "" H 3450 1700 50  0001 C CNN
 	1    3450 1700
@@
 Wire Wire Line
 	3550 1450 3300 1450
+$Comp
+L ROTARY-ENCODER ROT1
+U 1 1 59369A4E
+P 5700 5600
+F 0 "ROT1" H 5700 5850 60  0000 C CNN
+F 1 "ROTARY-ENCODER" H 5700 5320 60  0000 C CNN
+F 2 "sparkfun:SF-ROTARY-ENCODER" H 5700 5600 60  0001 C CNN
+F 3 "" H 5700 5600 60  0000 C CNN
+	1    5700 5600
+	-1   0    0    -1
+$EndComp
+Wire Wire Line
+	6050 5700 6300 5700
+Wire Wire Line
+	5100 5600 5350 5600
+Text Label 4700 5700 0    60   ~ 0
+ENC_B
+Text Label 4000 3500 0    60   ~ 0
+MCU_A
+Text Label 4000 3400 0    60   ~ 0
+MCU_B
+Wire Wire Line
+	3700 5200 7250 5200
+Wire Wire Line
+	3700 5200 3700 3200
+Wire Wire Line
+	3400 5500 3400 3500
+Wire Wire Line
+	3200 3400 3200 5700
+$Comp
+L R R6
+U 1 1 5936D3B1
+P 6950 5500
+F 0 "R6" V 7030 5500 50  0000 C CNN
+F 1 "27k" V 6950 5500 50  0000 C CNN
+F 2 "Resistors_SMD:R_0805_HandSoldering" V 6880 5500 50  0001 C CNN
+F 3 "" H 6950 5500 50  0001 C CNN
+	1    6950 5500
+	0    1    1    0
+$EndComp
+$Comp
+L R R4
+U 1 1 5936D489
+P 4350 5500
+F 0 "R4" V 4430 5500 50  0000 C CNN
+F 1 "27k" V 4350 5500 50  0000 C CNN
+F 2 "Resistors_SMD:R_0805_HandSoldering" V 4280 5500 50  0001 C CNN
+F 3 "" H 4350 5500 50  0001 C CNN
+	1    4350 5500
+	0    1    1    0
+$EndComp
+$Comp
+L R R5
+U 1 1 5936D4E2
+P 4350 5700
+F 0 "R5" V 4430 5700 50  0000 C CNN
+F 1 "27k" V 4350 5700 50  0000 C CNN
+F 2 "Resistors_SMD:R_0805_HandSoldering" V 4280 5700 50  0001 C CNN
+F 3 "" H 4350 5700 50  0001 C CNN
+	1    4350 5700
+	0    1    1    0
+$EndComp
+$Comp
+L C C5
+U 1 1 5936D604
+P 4100 5950
+F 0 "C5" H 4125 6050 50  0000 L CNN
+F 1 "100nF" H 4125 5850 50  0000 L CNN
+F 2 "Capacitors_SMD:C_0805_HandSoldering" H 4138 5800 50  0001 C CNN
+F 3 "" H 4100 5950 50  0001 C CNN
+	1    4100 5950
+	1    0    0    -1
+$EndComp
+$Comp
+L C C4
+U 1 1 5936D66B
+P 3750 5950
+F 0 "C4" H 3775 6050 50  0000 L CNN
+F 1 "100nF" H 3775 5850 50  0000 L CNN
+F 2 "Capacitors_SMD:C_0805_HandSoldering" H 3788 5800 50  0001 C CNN
+F 3 "" H 3750 5950 50  0001 C CNN
+	1    3750 5950
+	1    0    0    -1
+$EndComp
+$Comp
+L GND #PWR021
+U 1 1 5936D6C9
+P 4100 6200
+F 0 "#PWR021" H 4100 5950 50  0001 C CNN
+F 1 "GND" H 4100 6050 50  0000 C CNN
+F 2 "" H 4100 6200 50  0001 C CNN
+F 3 "" H 4100 6200 50  0001 C CNN
+	1    4100 6200
+	1    0    0    -1
+$EndComp
+$Comp
+L GND #PWR022
+U 1 1 5936D716
+P 3750 6200
+F 0 "#PWR022" H 3750 5950 50  0001 C CNN
+F 1 "GND" H 3750 6050 50  0000 C CNN
+F 2 "" H 3750 6200 50  0001 C CNN
+F 3 "" H 3750 6200 50  0001 C CNN
+	1    3750 6200
+	1    0    0    -1
+$EndComp
+Wire Wire Line
+	3750 6200 3750 6100
+Wire Wire Line
+	4100 6100 4100 6200
+Wire Wire Line
+	4100 5800 4100 5700
+Wire Wire Line
+	3200 5700 4200 5700
+Wire Wire Line
+	3400 5500 4200 5500
+Wire Wire Line
+	3750 5500 3750 5800
+Connection ~ 3750 5500
+Connection ~ 4100 5700
+Wire Wire Line
+	4500 5700 5350 5700
+Wire Wire Line
+	5350 5500 4500 5500
+Wire Wire Line
+	6050 5500 6800 5500
+Wire Wire Line
+	7100 5500 7250 5500
+Wire Wire Line
+	7250 5200 7250 5600
+Wire Wire Line
+	7250 5900 7250 6000
+Connection ~ 7250 5500
 $EndSCHEMATC
