File: shield/shield.kicad_pcb (KiCad board)
At the start: 2 copper layers, 25.7 x 34.4 mm, 23 parts, among them J1 Screw_Terminal_1x04, J2 Screw_Terminal_1x02, J4 Screw_Terminal_1x06, P1 CONN_01X08, P2 CONN_01X08, Q1 Q_NMOS_GSD, Q2 Q_NMOS_GSD, Q3 Q_NMOS_GSD, U1 LM1117-3.3

Commit message: Finished updating PCB to 2 layers
Parts:
- added ?: , custom_footprints:35-6-stitching-via, F.Cu at (144.8, 109.0)
- added ?: , custom_footprints:35-6-stitching-via, F.Cu at (147.8, 90.0)
- added ?: , custom_footprints:35-6-stitching-via, F.Cu at (148.0, 92.0)
- added ?: , custom_footprints:35-6-stitching-via, F.Cu at (151.2, 91.2)
- added ?: , custom_footprints:35-6-stitching-via, F.Cu at (151.5, 93.6)
- added ?: , custom_footprints:35-6-stitching-via, F.Cu at (151.2, 95.7)
- added ?: , custom_footprints:35-6-stitching-via, F.Cu at (151.1, 97.5)
- added ?: , custom_footprints:35-6-stitching-via, F.Cu at (145.8, 103.3)
- added ?: , custom_footprints:35-6-stitching-via, F.Cu at (143.4, 113.5)
- added ?: , custom_footprints:35-6-stitching-via, F.Cu at (143.3, 115.7)
- added ?: , custom_footprints:35-6-stitching-via, F.Cu at (149.9, 117.8)
- added ?: , custom_footprints:35-6-stitching-via, F.Cu at (143.5, 109.1)
- added ?: , custom_footprints:35-6-stitching-via, F.Cu at (144.8, 117.8)
- added ?: , custom_footprints:35-6-stitching-via, F.Cu at (151.5, 111.8)
- added ?: , custom_footprints:35-6-stitching-via, F.Cu at (153.3, 113.7)
- added ?: , custom_footprints:35-6-stitching-via, F.Cu at (151.4, 115.2)
- added ?: , custom_footprints:35-6-stitching-via, F.Cu at (153.1, 117.6)
- added ?: , custom_footprints:35-6-stitching-via, F.Cu at (149.3, 111.8)
- added ?: , custom_footprints:35-6-stitching-via, F.Cu at (131.6, 115.1)
- added ?: , custom_footprints:35-6-stitching-via, F.Cu at (141.9, 118.0)
- added ?: , custom_footprints:35-6-stitching-via, F.Cu at (140.0, 94.4)
- added ?: , custom_footprints:35-6-stitching-via, F.Cu at (144.2, 95.0)
- added ?: , custom_footprints:35-6-stitching-via, F.Cu at (147.9, 86.2)
- added ?: , custom_footprints:35-6-stitching-via, F.Cu at (150.7, 87.5)
- ?: moved to F.Cu
- moved ? 0.35 mm to (151.5, 88.8), turned to 0 degrees
Routing:
- net GND: track 6.23 -> 58.3 mm, vias 1 -> 3
- net /PIR_IN: track 23.5 -> 32.0 mm, vias 0 -> 2
- net Net-(Q2-Pad1): track 20.4 -> 27.1 mm, vias 1 -> 2
- net +12V: track 9.59 -> 5.89 mm
- net Net-(D1-Pad2): track 8.21 -> 6.78 mm
